Commit message: feat(robot,cad): scaffold setup
Signed-off-by: Mumtahin Farabi <mfarabi619@gmail.com>

File: apps/robot/urdf/robot.urdf (robot description, URDF)
Before this commit: robot robot, 5 links, 4 joints
Links:
- removed link body
- added link wheel_fl; visual mesh filename=package://robot/meshes/wheel_hub.stl scale=0.001 0.001 0.001; visual mesh filename=package://robot/meshes/wheel_rim.stl scale=0.001 0.001 0.001
- added link wheel_fr; visual mesh filename=package://robot/meshes/wheel_hub.stl scale=0.001 0.001 0.001; visual mesh filename=package://robot/meshes/wheel_rim.stl scale=0.001 0.001 0.001
- added link wheel_rl; visual mesh filename=package://robot/meshes/wheel_hub.stl scale=0.001 0.001 0.001; visual mesh filename=package://robot/meshes/wheel_rim.stl scale=0.001 0.001 0.001
- added link wheel_rr; visual mesh filename=package://robot/meshes/wheel_hub.stl scale=0.001 0.001 0.001; visual mesh filename=package://robot/meshes/wheel_rim.stl scale=0.001 0.001 0.001
- link chassis: geometry visual mesh filename=package://robot/meshes/chassis_aluminum.stl scale=0.001 0.001 0.001; visual mesh filename=package://robot/meshes/chassis_bracket.stl scale=0.001 0.001 0.001
Joints:
- removed joint base_to_body
- removed joint body_to_chassis
- added joint base_to_chassis: type fixed, parent base_link, child chassis, origin rpy=0 0 0
- added joint wheel_fl_joint: type continuous, parent chassis, child wheel_fl, origin xyz=0.53 0.527 0.178, axis 0 1 0
- added joint wheel_fr_joint: type continuous, parent chassis, child wheel_fr, origin xyz=0.53 -0.527 0.178, axis 0 1 0
- added joint wheel_rl_joint: type continuous, parent chassis, child wheel_rl, origin xyz=-0.53 0.527 0.178, axis 0 1 0
- added joint wheel_rr_joint: type continuous, parent chassis, child wheel_rr, origin xyz=-0.53 -0.527 0.178, axis 0 1 0
