Commit message: feat(robot): overhaul setup
Signed-off-by: Mumtahin Farabi <mfarabi619@gmail.com>

File: apps/robot/urdf/robot.urdf (robot description, URDF)
Before this commit: robot robot, 8 links, 7 joints
Links:
- added link base_footprint
- added link motor_fl; visual mesh filename=package://robot/meshes/motor_fl.dae
- added link motor_fr; visual mesh filename=package://robot/meshes/motor_fr.dae
- added link motor_rl; visual mesh filename=package://robot/meshes/motor_rl.dae
- added link motor_rr; visual mesh filename=package://robot/meshes/motor_rr.dae
- added link mount_fl, mass 0.2518; visual mesh filename=package://robot/meshes/mount_fl.dae
- added link mount_fr, mass 0.2518; visual mesh filename=package://robot/meshes/mount_fr.dae
- added link mount_rl, mass 0.2518; visual mesh filename=package://robot/meshes/mount_rl.dae
- added link mount_rr, mass 0.2518; visual mesh filename=package://robot/meshes/mount_rr.dae
- link camera_link: geometry visual mesh filename=package://robot/meshes/camera_link.dae
- link chassis: mass None -> 41.2746; geometry collision box size=1.1500 1.0000 0.0254; visual mesh filename=package://robot/meshes/chassis.dae
- link wheel_fl: mass None -> 5.2861; geometry collision cylinder length=0.1000 radius=0.1749; visual mesh filename=package://robot/meshes/wheel_fl.dae
- link wheel_fr: mass None -> 5.2861; geometry collision cylinder length=0.1000 radius=0.1749; visual mesh filename=package://robot/meshes/wheel_fr.dae
- link wheel_rl: mass None -> 5.2861; geometry collision cylinder length=0.1000 radius=0.1749; visual mesh filename=package://robot/meshes/wheel_rl.dae
- link wheel_rr: mass None -> 5.2861; geometry collision cylinder length=0.1000 radius=0.1749; visual mesh filename=package://robot/meshes/wheel_rr.dae
Joints:
- removed joint base_to_camera
- removed joint base_to_chassis
- removed joint camera_to_optical
- added joint base_footprint_joint: type fixed, parent base_link, child base_footprint, origin xyz=0.0000 0.0000 0.0264 rpy=0.0000 0.0000 0.0000
- added joint camera_mount_joint: type fixed, parent chassis, child camera_link, origin xyz=0.5600 0.0000 0.3000 rpy=0.0000 0.0000 0.0000
- added joint camera_optical_joint: type fixed, parent camera_link, child camera_optical_frame, origin xyz=0.0000 0.0000 0.0000 rpy=-1.5708 0.0000 -1.5708
- added joint chassis_joint: type fixed, parent base_link, child chassis, origin xyz=0.0000 0.0000 0.0000 rpy=0.0000 0.0000 0.0000
- added joint motor_fl_joint: type fixed, parent mount_fl, child motor_fl, origin xyz=-0.0260 0.0660 -0.0732 rpy=0.0000 0.0000 0.0000
- added joint motor_fr_joint: type fixed, parent mount_fr, child motor_fr, origin xyz=-0.0260 -0.0660 -0.0732 rpy=0.0000 0.0000 0.0000
- added joint motor_rl_joint: type fixed, parent mount_rl, child motor_rl, origin xyz=-0.0260 0.0660 -0.0732 rpy=0.0000 0.0000 0.0000
- added joint motor_rr_joint: type fixed, parent mount_rr, child motor_rr, origin xyz=-0.0260 -0.0660 -0.0732 rpy=0.0000 0.0000 0.0000
- added joint mount_fl_joint: type fixed, parent chassis, child mount_fl, origin xyz=0.4000 0.4742 0.2746 rpy=0.0000 0.0000 0.0000
- added joint mount_fr_joint: type fixed, parent chassis, child mount_fr, origin xyz=0.4000 -0.4742 0.2746 rpy=0.0000 0.0000 0.0000
- added joint mount_rl_joint: type fixed, parent chassis, child mount_rl, origin xyz=-0.4000 0.4742 0.2746 rpy=0.0000 0.0000 0.0000
- added joint mount_rr_joint: type fixed, parent chassis, child mount_rr, origin xyz=-0.4000 -0.4742 0.2746 rpy=0.0000 0.0000 0.0000
- joint wheel_fl_joint: axis 0 1 0 -> 0.0 1.0 0.0; origin xyz=0.53 0.527 0.178 -> xyz=0.0000 0.0450 0.0000 rpy=0.0000 0.0000 0.0000; parent chassis -> motor_fl
- joint wheel_fr_joint: axis 0 1 0 -> 0.0 1.0 0.0; origin xyz=0.53 -0.527 0.178 -> xyz=0.0000 -0.0450 0.0000 rpy=0.0000 0.0000 0.0000; parent chassis -> motor_fr
- joint wheel_rl_joint: axis 0 1 0 -> 0.0 1.0 0.0; origin xyz=-0.53 0.527 0.178 -> xyz=0.0000 0.0450 0.0000 rpy=0.0000 0.0000 0.0000; parent chassis -> motor_rl
- joint wheel_rr_joint: axis 0 1 0 -> 0.0 1.0 0.0; origin xyz=-0.53 -0.527 0.178 -> xyz=0.0000 -0.0450 0.0000 rpy=0.0000 0.0000 0.0000; parent chassis -> motor_rr
