Commit message: feat(robot): overhaul setup
Signed-off-by: Mumtahin Farabi <mfarabi619@gmail.com>

File: apps/robot/urdf/robot.urdf.xacro (robot description, xacro)
@@ -1,4 +1,4 @@
 <?xml version="1.0"?>
-<robot name="robot">
+<robot name="robot" xmlns:xacro="http://www.ros.org/wiki/xacro">
   <material name="aluminum"><color rgba="0.78 0.80 0.83 1.0"/></material>
   <material name="plywood"><color rgba="0.78 0.62 0.40 1.0"/></material>
@@ -84,3 +84,20 @@
     <origin rpy="-1.5707963 0 -1.5707963"/>
   </joint>
+  <xacro:macro name="wheel_ros2_control_joint" params="name">
+    <joint name="${name}">
+      <command_interface name="velocity"/>
+      <state_interface name="position"/>
+      <state_interface name="velocity"/>
+    </joint>
+  </xacro:macro>
+  <ros2_control name="RobotSystem" type="system">
+    <hardware>
+      <plugin>mock_components/GenericSystem</plugin>
+      <param name="calculate_dynamics">true</param>
+    </hardware>
+    <xacro:wheel_ros2_control_joint name="wheel_fl_joint"/>
+    <xacro:wheel_ros2_control_joint name="wheel_fr_joint"/>
+    <xacro:wheel_ros2_control_joint name="wheel_rl_joint"/>
+    <xacro:wheel_ros2_control_joint name="wheel_rr_joint"/>
+  </ros2_control>
 </robot>
