Commit message: feat(robot): overhaul setup
Signed-off-by: Mumtahin Farabi <mfarabi619@gmail.com>

File: apps/robot/robot_description/urdf/robot.sim.urdf (robot description, URDF)
Before this commit: robot robot, 20 links, 19 joints
Links:
- removed link camera_link
- removed link camera_optical_frame
- added link camera_0_color_optical_frame
- added link camera_0_link
- added link camera_1_color_optical_frame
- added link camera_1_link
Joints:
- removed joint camera_link_joint
- removed joint camera_optical_frame_joint
- added joint camera_0_color_optical_frame_joint: type fixed, parent camera_0_link, child camera_0_color_optical_frame, origin xyz=0.0000 0.0000 0.0000 rpy=-1.5708 0.0000 -1.5708
- added joint camera_0_link_joint: type fixed, parent camera_mount_link, child camera_0_link, origin xyz=0.0000 0.0000 0.0000 rpy=0.0000 0.3100 0.0000
- added joint camera_1_color_optical_frame_joint: type fixed, parent camera_1_link, child camera_1_color_optical_frame, origin xyz=0.0000 0.0000 0.0000 rpy=-1.5708 0.0000 -1.5708
- added joint camera_1_link_joint: type fixed, parent camera_mount_link, child camera_1_link, origin xyz=0.0000 0.0000 0.0000 rpy=0.0000 0.3100 0.0000

File: apps/robot/robot_description/urdf/robot.urdf (robot description, URDF)
Before this commit: robot robot, 20 links, 19 joints
Links:
- removed link camera_link
- removed link camera_optical_frame
- added link camera_0_color_optical_frame
- added link camera_0_link
- added link camera_1_color_optical_frame
- added link camera_1_link
Joints:
- removed joint camera_link_joint
- removed joint camera_optical_frame_joint
- added joint camera_0_color_optical_frame_joint: type fixed, parent camera_0_link, child camera_0_color_optical_frame, origin xyz=0.0000 0.0000 0.0000 rpy=-1.5708 0.0000 -1.5708
- added joint camera_0_link_joint: type fixed, parent camera_mount_link, child camera_0_link, origin xyz=0.0000 0.0000 0.0000 rpy=0.0000 0.3100 0.0000
- added joint camera_1_color_optical_frame_joint: type fixed, parent camera_1_link, child camera_1_color_optical_frame, origin xyz=0.0000 0.0000 0.0000 rpy=-1.5708 0.0000 -1.5708
- added joint camera_1_link_joint: type fixed, parent camera_mount_link, child camera_1_link, origin xyz=0.0000 0.0000 0.0000 rpy=0.0000 0.3100 0.0000

Commit message: feat(robot): overhaul setup
Signed-off-by: Mumtahin Farabi <mfarabi619@gmail.com>

File: apps/robot/robot_description/urdf/robot.sim.urdf (robot description, URDF)
Before this commit: robot robot, 22 links, 21 joints
Links:
- added link ptu_0_base_link
- added link ptu_0_pan_link, mass 0.0100
- added link ptu_0_tilt_link, mass 0.0100
Joints:
- added joint ptu_0_base_link_joint: type fixed, parent camera_mount_link, child ptu_0_base_link, origin xyz=0.0000 0.0000 0.0000 rpy=0.0000 0.0000 0.0000
- added joint ptu_0_pan: type revolute, parent ptu_0_base_link, child ptu_0_pan_link, origin xyz=0.0000 0.0000 0.0000 rpy=0.0000 0.0000 0.0000, axis 0 0 1, limit lower=-1.5708 upper=1.5708 effort=1.0 velocity=3.1416
- added joint ptu_0_tilt: type revolute, parent ptu_0_pan_link, child ptu_0_tilt_link, origin xyz=0.0000 0.0000 0.0000 rpy=0.0000 0.0000 0.0000, axis 0 1 0, limit lower=-1.5708 upper=1.5708 effort=1.0 velocity=3.1416
- joint camera_0_link_joint: origin xyz=0.0000 0.0000 0.0000 rpy=0.0000 0.3100 0.0000 -> xyz=-0.5750 0.0000 0.7500 rpy=0.0000 0.3100 0.0000; parent camera_mount_link -> base_link
- joint camera_1_link_joint: origin xyz=0.0000 0.0000 0.0000 rpy=0.0000 0.3100 0.0000 -> xyz=0.4050 0.4746 0.5000 rpy=0.0000 0.3100 0.0000; parent camera_mount_link -> base_link

File: apps/robot/robot_description/urdf/robot.urdf (robot description, URDF)
Before this commit: robot robot, 22 links, 21 joints
Links:
- added link ptu_0_base_link
- added link ptu_0_pan_link, mass 0.0100
- added link ptu_0_tilt_link, mass 0.0100
Joints:
- added joint ptu_0_base_link_joint: type fixed, parent camera_mount_link, child ptu_0_base_link, origin xyz=0.0000 0.0000 0.0000 rpy=0.0000 0.0000 0.0000
- added joint ptu_0_pan: type revolute, parent ptu_0_base_link, child ptu_0_pan_link, origin xyz=0.0000 0.0000 0.0000 rpy=0.0000 0.0000 0.0000, axis 0 0 1, limit lower=-1.5708 upper=1.5708 effort=1.0 velocity=3.1416
- added joint ptu_0_tilt: type revolute, parent ptu_0_pan_link, child ptu_0_tilt_link, origin xyz=0.0000 0.0000 0.0000 rpy=0.0000 0.0000 0.0000, axis 0 1 0, limit lower=-1.5708 upper=1.5708 effort=1.0 velocity=3.1416
- joint camera_0_link_joint: origin xyz=0.0000 0.0000 0.0000 rpy=0.0000 0.3100 0.0000 -> xyz=-0.5750 0.0000 0.7500 rpy=0.0000 0.3100 0.0000; parent camera_mount_link -> base_link
- joint camera_1_link_joint: origin xyz=0.0000 0.0000 0.0000 rpy=0.0000 0.3100 0.0000 -> xyz=0.4050 0.4746 0.5000 rpy=0.0000 0.3100 0.0000; parent camera_mount_link -> base_link
