Commit message: feat(robot): overhaul setup
Signed-off-by: Mumtahin Farabi <mfarabi619@gmail.com>

File: apps/robot/description/urdf/robot0/robot.urdf (robot description, URDF)
Before this commit: robot robot, 22 links, 21 joints
Links:
- removed link camera_1_color_optical_frame
- removed link camera_1_link
Joints:
- removed joint camera_1_color_optical_frame_joint
- removed joint camera_1_link_joint

File: apps/robot/description/urdf/robot4/robot.sim.urdf (robot description, URDF)
Before this commit: robot robot, 20 links, 19 joints
Links:
- removed link camera_mount_link
- removed link imu_0_link
- link camera_0_link: geometry 
Joints:
- removed joint camera_mount_link_joint
- removed joint imu_0_link_joint
- joint camera_0_link_joint: origin xyz=0.5750 0.5000 0.3100 rpy=0.0000 0.3100 0.0000 -> xyz=0.5750 0.5000 0.3100 rpy=0.0000 0.0000 0.0000

File: apps/robot/description/urdf/robot4/robot.urdf (robot description, URDF)
Before this commit: robot robot, 20 links, 19 joints
Links:
- removed link camera_mount_link
- removed link imu_0_link
- link camera_0_link: geometry 
Joints:
- removed joint camera_mount_link_joint
- removed joint imu_0_link_joint
- joint camera_0_link_joint: origin xyz=0.5750 0.5000 0.3100 rpy=0.0000 0.3100 0.0000 -> xyz=0.5750 0.5000 0.3100 rpy=0.0000 0.0000 0.0000

File: apps/robot/description/urdf/robot5/robot.sim.urdf (robot description, URDF)
Before this commit: robot robot, 20 links, 19 joints
Links:
- removed link camera_mount_link
- removed link imu_0_link
- link camera_0_link: geometry 
Joints:
- removed joint camera_mount_link_joint
- removed joint imu_0_link_joint
- joint camera_0_link_joint: origin xyz=0.5750 0.5000 0.3100 rpy=0.0000 0.3100 0.0000 -> xyz=0.5750 0.5000 0.3100 rpy=0.0000 0.0000 0.0000
