Commit message: feat(robot): overhaul setup
Signed-off-by: Mumtahin Farabi <mfarabi619@gmail.com>

File: apps/robot/description/urdf/robot0/robot.sim.urdf (robot description, URDF)
Before this commit: robot robot, 23 links, 22 joints
Links:
- removed link gps_link
- added link lidar_link
Joints:
- removed joint gps_link_joint
- added joint lidar_link_joint: type fixed, parent base_link, child lidar_link, origin xyz=0.0000 0.0000 0.4000 rpy=0.0000 0.0000 0.0000

File: apps/robot/description/urdf/robot0/robot.urdf (robot description, URDF)
Before this commit: robot robot, 23 links, 22 joints
Links:
- removed link gps_link
Joints:
- removed joint gps_link_joint

File: apps/robot/description/urdf/robot1/robot.sim.urdf (robot description, URDF)
Before this commit: robot robot, 16 links, 15 joints
Links:
- added link lidar_link
Joints:
- added joint lidar_link_joint: type fixed, parent base_link, child lidar_link, origin xyz=0.0000 0.0000 0.4000 rpy=0.0000 0.0000 0.0000

Commit message: feat(robot/description): overhaul setup
Signed-off-by: Mumtahin Farabi <mfarabi619@gmail.com>

File: apps/robot/description/urdf/robot0/robot.sim.urdf (robot description, URDF)
Before this commit: robot robot, 23 links, 22 joints
Links:
- removed link lidar_link
Joints:
- removed joint lidar_link_joint
- joint camera_1_link_joint: origin xyz=0.4050 0.4746 0.5000 rpy=0.0000 0.3100 0.0000 -> xyz=0.5750 0.5000 0.3100 rpy=0.0000 0.3100 0.0000

File: apps/robot/description/urdf/robot0/robot.urdf (robot description, URDF)
Before this commit: robot robot, 22 links, 21 joints
Joints:
- joint camera_1_link_joint: origin xyz=0.4050 0.4746 0.5000 rpy=0.0000 0.3100 0.0000 -> xyz=0.5750 0.5000 0.3100 rpy=0.0000 0.3100 0.0000

File: apps/robot/description/urdf/robot1/robot.sim.urdf (robot description, URDF)
Before this commit: robot robot, 17 links, 16 joints
Links:
- removed link lidar_link
- added link camera_0_color_optical_frame
- added link camera_0_link; visual mesh filename=package://robot_description/meshes/orbbec_gemini_335l.dae
Joints:
- removed joint lidar_link_joint
- added joint camera_0_color_optical_frame_joint: type fixed, parent camera_0_link, child camera_0_color_optical_frame, origin xyz=0.0000 0.0000 0.0000 rpy=-1.5708 0.0000 -1.5708
- added joint camera_0_link_joint: type fixed, parent base_link, child camera_0_link, origin xyz=0.5750 0.5000 0.3100 rpy=0.0000 0.0000 0.0000

File: apps/robot/description/urdf/robot1/robot.urdf (robot description, URDF)
Before this commit: robot robot, 16 links, 15 joints
Links:
- added link camera_0_color_optical_frame
- added link camera_0_link; visual mesh filename=package://robot_description/meshes/orbbec_gemini_335l.dae
Joints:
- added joint camera_0_color_optical_frame_joint: type fixed, parent camera_0_link, child camera_0_color_optical_frame, origin xyz=0.0000 0.0000 0.0000 rpy=-1.5708 0.0000 -1.5708
- added joint camera_0_link_joint: type fixed, parent base_link, child camera_0_link, origin xyz=0.5750 0.5000 0.3100 rpy=0.0000 0.0000 0.0000

File: apps/robot/description/urdf/robot2/robot.sim.urdf (robot description, URDF)
Before this commit: robot robot, 17 links, 16 joints
Links:
- removed link lidar_link
Joints:
- removed joint lidar_link_joint
