Commit message: feat(robot/{description,generator_common,simulator): overhaul setup
Signed-off-by: Mumtahin Farabi <mfarabi619@gmail.com>

File: apps/robot/description/urdf/robot0/robot.sim.urdf (robot description, URDF)
Before this commit: robot robot, 20 links, 19 joints
Links:
- removed link camera_mount_link
- removed link front_left_motor_link
- removed link front_left_mount_link
- removed link front_left_wheel_link
- removed link front_right_motor_link
- removed link front_right_mount_link
- removed link front_right_wheel_link
- removed link imu_0_link
- added link front_left_caster_link; collision sphere radius=0.1396
- added link front_right_caster_link; collision sphere radius=0.1396
- link camera_0_link: geometry 
- link chassis: geometry collision box size=1.2192 1.0000 0.0254; visual mesh filename=package://robot_description/meshes/robot0/chassis.dae
- link inertial_link: mass 41.2746 -> 63.6981
- link rear_left_motor_link: geometry visual mesh filename=package://robot_description/meshes/robot0/rear_left_motor_l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
- link rear_left_mount_link: geometry visual mesh filename=package://robot_description/meshes/robot0/rear_left_mount_l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
- link rear_left_wheel_link: geometry collision cylinder length=0.1000 radius=0.1749; visual mesh filename=package://robot_description/meshes/robot0/rear_left_wheel_l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
- link rear_right_motor_link: geometry visual mesh filename=package://robot_description/meshes/robot0/rear_right_motor_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
- link rear_right_mount_link: geometry visual mesh filename=package://robot_description/meshes/robot0/rear_right_mount_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
- link rear_right_wheel_link: geometry collision cylinder length=0.1000 radius=0.1749; visual mesh filename=package://robot_description/meshes/robot0/rear_right_wheel_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
Joints:
- removed joint camera_mount_link_joint
- removed joint front_left_motor_joint
- removed joint front_left_mount_joint
- removed joint front_left_wheel_joint
- removed joint front_right_motor_joint
- removed joint front_right_mount_joint
- removed joint front_right_wheel_joint
- removed joint imu_0_link_joint
- added joint front_left_caster_joint: type fixed, parent chassis, child front_left_caster_link, origin xyz=0.4682 0.5508 0.1222 rpy=0.0000 0.0000 0.0000
- added joint front_right_caster_joint: type fixed, parent chassis, child front_right_caster_link, origin xyz=0.4682 -0.5508 0.1222 rpy=0.0000 0.0000 0.0000
- joint camera_0_link_joint: origin xyz=0.5750 0.5000 0.3100 rpy=0.0000 0.3100 0.0000 -> xyz=0.5300 0.4750 0.5660 rpy=0.0000 0.0000 0.0000
- joint rear_left_mount_joint: origin xyz=-0.4000 0.4742 0.2746 rpy=0.0000 0.0000 0.0000 -> xyz=-0.5246 0.4742 0.2746 rpy=0.0000 0.0000 0.0000
- joint rear_right_mount_joint: origin xyz=-0.4000 -0.4742 0.2746 rpy=0.0000 0.0000 0.0000 -> xyz=-0.5246 -0.4742 0.2746 rpy=0.0000 0.0000 0.0000

File: apps/robot/description/urdf/robot0/robot.urdf (robot description, URDF)
Before this commit: robot robot, 20 links, 19 joints
Links:
- removed link camera_mount_link
- removed link front_left_motor_link
- removed link front_left_mount_link
- removed link front_left_wheel_link
- removed link front_right_motor_link
- removed link front_right_mount_link
- removed link front_right_wheel_link
- removed link imu_0_link
- added link front_left_caster_link; collision sphere radius=0.1396
- added link front_right_caster_link; collision sphere radius=0.1396
- link camera_0_link: geometry 
- link chassis: geometry collision box size=1.2192 1.0000 0.0254; visual mesh filename=package://robot_description/meshes/robot0/chassis.dae
- link inertial_link: mass 41.2746 -> 63.6981
- link rear_left_motor_link: geometry visual mesh filename=package://robot_description/meshes/robot0/rear_left_motor_l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
- link rear_left_mount_link: geometry visual mesh filename=package://robot_description/meshes/robot0/rear_left_mount_l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
- link rear_left_wheel_link: geometry collision cylinder length=0.1000 radius=0.1749; visual mesh filename=package://robot_description/meshes/robot0/rear_left_wheel_l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
- link rear_right_motor_link: geometry visual mesh filename=package://robot_description/meshes/robot0/rear_right_motor_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
- link rear_right_mount_link: geometry visual mesh filename=package://robot_description/meshes/robot0/rear_right_mount_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
- link rear_right_wheel_link: geometry collision cylinder length=0.1000 radius=0.1749; visual mesh filename=package://robot_description/meshes/robot0/rear_right_wheel_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
Joints:
- removed joint camera_mount_link_joint
- removed joint front_left_motor_joint
- removed joint front_left_mount_joint
- removed joint front_left_wheel_joint
- removed joint front_right_motor_joint
- removed joint front_right_mount_joint
- removed joint front_right_wheel_joint
- removed joint imu_0_link_joint
- added joint front_left_caster_joint: type fixed, parent chassis, child front_left_caster_link, origin xyz=0.4682 0.5508 0.1222 rpy=0.0000 0.0000 0.0000
- added joint front_right_caster_joint: type fixed, parent chassis, child front_right_caster_link, origin xyz=0.4682 -0.5508 0.1222 rpy=0.0000 0.0000 0.0000
- joint camera_0_link_joint: origin xyz=0.5750 0.5000 0.3100 rpy=0.0000 0.3100 0.0000 -> xyz=0.5300 0.4750 0.5660 rpy=0.0000 0.0000 0.0000
- joint rear_left_mount_joint: origin xyz=-0.4000 0.4742 0.2746 rpy=0.0000 0.0000 0.0000 -> xyz=-0.5246 0.4742 0.2746 rpy=0.0000 0.0000 0.0000
- joint rear_right_mount_joint: origin xyz=-0.4000 -0.4742 0.2746 rpy=0.0000 0.0000 0.0000 -> xyz=-0.5246 -0.4742 0.2746 rpy=0.0000 0.0000 0.0000

File: apps/robot/description/urdf/robot1/robot.sim.urdf (robot description, URDF)
Before this commit: robot robot, 18 links, 17 joints
Links:
- removed link front_left_motor_link
- removed link front_left_mount_link
- removed link front_left_wheel_link
- removed link front_right_motor_link
- removed link front_right_mount_link
- removed link front_right_wheel_link
- added link front_left_caster_link; collision sphere radius=0.1396
- added link front_right_caster_link; collision sphere radius=0.1396
- link camera_0_link: geometry 
- link chassis: geometry collision box size=0.7500 0.4000 0.0254; visual mesh filename=package://robot_description/meshes/robot1/chassis.dae
- link inertial_link: mass 41.2746 -> 32.6186
- link rear_left_motor_link: geometry visual mesh filename=package://robot_description/meshes/robot1/rear_left_motor_l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
- link rear_left_mount_link: geometry visual mesh filename=package://robot_description/meshes/robot1/rear_left_mount_l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
- link rear_left_wheel_link: geometry collision cylinder length=0.1000 radius=0.1749; visual mesh filename=package://robot_description/meshes/robot1/rear_left_wheel_l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
- link rear_right_motor_link: geometry visual mesh filename=package://robot_description/meshes/robot1/rear_right_motor_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
- link rear_right_mount_link: geometry visual mesh filename=package://robot_description/meshes/robot1/rear_right_mount_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
- link rear_right_wheel_link: geometry collision cylinder length=0.1000 radius=0.1749; visual mesh filename=package://robot_description/meshes/robot1/rear_right_wheel_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
Joints:
- removed joint front_left_motor_joint
- removed joint front_left_mount_joint
- removed joint front_left_wheel_joint
- removed joint front_right_motor_joint
- removed joint front_right_mount_joint
- removed joint front_right_wheel_joint
- added joint front_left_caster_joint: type fixed, parent chassis, child front_left_caster_link, origin xyz=0.2337 0.2508 0.1222 rpy=0.0000 0.0000 0.0000
- added joint front_right_caster_joint: type fixed, parent chassis, child front_right_caster_link, origin xyz=0.2337 -0.2508 0.1222 rpy=0.0000 0.0000 0.0000
- joint camera_0_link_joint: origin xyz=0.5750 0.5000 0.3100 rpy=0.0000 0.0000 0.0000 -> xyz=0.3500 0.0000 0.3600 rpy=0.0000 0.0000 0.0000
- joint rear_left_mount_joint: origin xyz=-0.4000 0.4742 0.2746 rpy=0.0000 0.0000 0.0000 -> xyz=-0.2400 0.1742 0.2746 rpy=0.0000 0.0000 0.0000
- joint rear_right_mount_joint: origin xyz=-0.4000 -0.4742 0.2746 rpy=0.0000 0.0000 0.0000 -> xyz=-0.2400 -0.1742 0.2746 rpy=0.0000 0.0000 0.0000

File: apps/robot/description/urdf/robot1/robot.urdf (robot description, URDF)
Before this commit: robot robot, 18 links, 17 joints
Links:
- removed link front_left_motor_link
- removed link front_left_mount_link
- removed link front_left_wheel_link
- removed link front_right_motor_link
- removed link front_right_mount_link
- removed link front_right_wheel_link
- added link front_left_caster_link; collision sphere radius=0.1396
- added link front_right_caster_link; collision sphere radius=0.1396
- link camera_0_link: geometry 
- link chassis: geometry collision box size=0.7500 0.4000 0.0254; visual mesh filename=package://robot_description/meshes/robot1/chassis.dae
- link inertial_link: mass 41.2746 -> 32.6186
- link rear_left_motor_link: geometry visual mesh filename=package://robot_description/meshes/robot1/rear_left_motor_l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
- link rear_left_mount_link: geometry visual mesh filename=package://robot_description/meshes/robot1/rear_left_mount_l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
- link rear_left_wheel_link: geometry collision cylinder length=0.1000 radius=0.1749; visual mesh filename=package://robot_description/meshes/robot1/rear_left_wheel_l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
- link rear_right_motor_link: geometry visual mesh filename=package://robot_description/meshes/robot1/rear_right_motor_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
- link rear_right_mount_link: geometry visual mesh filename=package://robot_description/meshes/robot1/rear_right_mount_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
- link rear_right_wheel_link: geometry collision cylinder length=0.1000 radius=0.1749; visual mesh filename=package://robot_description/meshes/robot1/rear_right_wheel_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
Joints:
- removed joint front_left_motor_joint
- removed joint front_left_mount_joint
- removed joint front_left_wheel_joint
- removed joint front_right_motor_joint
- removed joint front_right_mount_joint
- removed joint front_right_wheel_joint
- added joint front_left_caster_joint: type fixed, parent chassis, child front_left_caster_link, origin xyz=0.2337 0.2508 0.1222 rpy=0.0000 0.0000 0.0000
- added joint front_right_caster_joint: type fixed, parent chassis, child front_right_caster_link, origin xyz=0.2337 -0.2508 0.1222 rpy=0.0000 0.0000 0.0000
- joint camera_0_link_joint: origin xyz=0.5750 0.5000 0.3100 rpy=0.0000 0.0000 0.0000 -> xyz=0.3500 0.0000 0.3600 rpy=0.0000 0.0000 0.0000
- joint rear_left_mount_joint: origin xyz=-0.4000 0.4742 0.2746 rpy=0.0000 0.0000 0.0000 -> xyz=-0.2400 0.1742 0.2746 rpy=0.0000 0.0000 0.0000
- joint rear_right_mount_joint: origin xyz=-0.4000 -0.4742 0.2746 rpy=0.0000 0.0000 0.0000 -> xyz=-0.2400 -0.1742 0.2746 rpy=0.0000 0.0000 0.0000

File: apps/robot/description/urdf/robot2/robot.sim.urdf (robot description, URDF)
Before this commit: robot robot, 16 links, 15 joints
Links:
- removed link front_left_motor_link
- removed link front_left_mount_link
- removed link front_left_wheel_link
- removed link front_right_motor_link
- removed link front_right_mount_link
- removed link front_right_wheel_link
- added link camera_0_color_optical_frame
- added link camera_0_link
- added link front_left_caster_link; collision sphere radius=0.1396
- added link front_right_caster_link; collision sphere radius=0.1396
- link chassis: geometry collision box size=1.2192 1.0000 0.0254; visual mesh filename=package://robot_description/meshes/robot2/chassis.dae
- link inertial_link: mass 41.2746 -> 63.6981
- link rear_left_motor_link: geometry visual mesh filename=package://robot_description/meshes/robot2/rear_left_motor_l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
- link rear_left_mount_link: geometry visual mesh filename=package://robot_description/meshes/robot2/rear_left_mount_l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
- link rear_left_wheel_link: geometry collision cylinder length=0.1000 radius=0.1749; visual mesh filename=package://robot_description/meshes/robot2/rear_left_wheel_l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
- link rear_right_motor_link: geometry visual mesh filename=package://robot_description/meshes/robot2/rear_right_motor_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
- link rear_right_mount_link: geometry visual mesh filename=package://robot_description/meshes/robot2/rear_right_mount_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
- link rear_right_wheel_link: geometry collision cylinder length=0.1000 radius=0.1749; visual mesh filename=package://robot_description/meshes/robot2/rear_right_wheel_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
Joints:
- removed joint front_left_motor_joint
- removed joint front_left_mount_joint
- removed joint front_left_wheel_joint
- removed joint front_right_motor_joint
- removed joint front_right_mount_joint
- removed joint front_right_wheel_joint
- added joint camera_0_color_optical_frame_joint: type fixed, parent camera_0_link, child camera_0_color_optical_frame, origin xyz=0.0000 0.0000 0.0000 rpy=-1.5708 0.0000 -1.5708
- added joint camera_0_link_joint: type fixed, parent base_link, child camera_0_link, origin xyz=0.0000 0.0000 0.1000 rpy=0.0000 0.0000 0.0000
- added joint front_left_caster_joint: type fixed, parent chassis, child front_left_caster_link, origin xyz=0.4682 0.5508 0.1222 rpy=0.0000 0.0000 0.0000
- added joint front_right_caster_joint: type fixed, parent chassis, child front_right_caster_link, origin xyz=0.4682 -0.5508 0.1222 rpy=0.0000 0.0000 0.0000
- joint rear_left_mount_joint: origin xyz=-0.4000 0.4742 0.2746 rpy=0.0000 0.0000 0.0000 -> xyz=-0.5246 0.4742 0.2746 rpy=0.0000 0.0000 0.0000
- joint rear_right_mount_joint: origin xyz=-0.4000 -0.4742 0.2746 rpy=0.0000 0.0000 0.0000 -> xyz=-0.5246 -0.4742 0.2746 rpy=0.0000 0.0000 0.0000

File: apps/robot/description/urdf/robot2/robot.urdf (robot description, URDF)
Before this commit: robot robot, 16 links, 15 joints
Links:
- removed link front_left_motor_link
- removed link front_left_mount_link
- removed link front_left_wheel_link
- removed link front_right_motor_link
- removed link front_right_mount_link
- removed link front_right_wheel_link
- added link camera_0_color_optical_frame
- added link camera_0_link
- added link front_left_caster_link; collision sphere radius=0.1396
- added link front_right_caster_link; collision sphere radius=0.1396
- link chassis: geometry collision box size=1.2192 1.0000 0.0254; visual mesh filename=package://robot_description/meshes/robot2/chassis.dae
- link inertial_link: mass 41.2746 -> 63.6981
- link rear_left_motor_link: geometry visual mesh filename=package://robot_description/meshes/robot2/rear_left_motor_l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
- link rear_left_mount_link: geometry visual mesh filename=package://robot_description/meshes/robot2/rear_left_mount_l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
- link rear_left_wheel_link: geometry collision cylinder length=0.1000 radius=0.1749; visual mesh filename=package://robot_description/meshes/robot2/rear_left_wheel_l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
- link rear_right_motor_link: geometry visual mesh filename=package://robot_description/meshes/robot2/rear_right_motor_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
- link rear_right_mount_link: geometry visual mesh filename=package://robot_description/meshes/robot2/rear_right_mount_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
- link rear_right_wheel_link: geometry collision cylinder length=0.1000 radius=0.1749; visual mesh filename=package://robot_description/meshes/robot2/rear_right_wheel_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
Joints:
- removed joint front_left_motor_joint
- removed joint front_left_mount_joint
- removed joint front_left_wheel_joint
- removed joint front_right_motor_joint
- removed joint front_right_mount_joint
- removed joint front_right_wheel_joint
- added joint camera_0_color_optical_frame_joint: type fixed, parent camera_0_link, child camera_0_color_optical_frame, origin xyz=0.0000 0.0000 0.0000 rpy=-1.5708 0.0000 -1.5708
- added joint camera_0_link_joint: type fixed, parent base_link, child camera_0_link, origin xyz=0.0000 0.0000 0.1000 rpy=0.0000 0.0000 0.0000
- added joint front_left_caster_joint: type fixed, parent chassis, child front_left_caster_link, origin xyz=0.4682 0.5508 0.1222 rpy=0.0000 0.0000 0.0000
- added joint front_right_caster_joint: type fixed, parent chassis, child front_right_caster_link, origin xyz=0.4682 -0.5508 0.1222 rpy=0.0000 0.0000 0.0000
- joint rear_left_mount_joint: origin xyz=-0.4000 0.4742 0.2746 rpy=0.0000 0.0000 0.0000 -> xyz=-0.5246 0.4742 0.2746 rpy=0.0000 0.0000 0.0000
- joint rear_right_mount_joint: origin xyz=-0.4000 -0.4742 0.2746 rpy=0.0000 0.0000 0.0000 -> xyz=-0.5246 -0.4742 0.2746 rpy=0.0000 0.0000 0.0000

File: apps/robot/description/urdf/robot3/robot.sim.urdf (robot description, URDF)
Before this commit: robot robot, 18 links, 17 joints
Links:
- removed link front_left_motor_link
- removed link front_left_mount_link
- removed link front_left_wheel_link
- removed link front_right_motor_link
- removed link front_right_mount_link
- removed link front_right_wheel_link
- added link camera_mount_link
- added link front_left_caster_link; collision sphere radius=0.1396
- added link front_right_caster_link; collision sphere radius=0.1396
- added link imu_0_link
- link chassis: geometry collision box size=1.2192 1.0000 0.0254; visual mesh filename=package://robot_description/meshes/robot3/chassis.dae
- link inertial_link: mass 41.2746 -> 63.6981
- link rear_left_motor_link: geometry visual mesh filename=package://robot_description/meshes/robot3/rear_left_motor_l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
- link rear_left_mount_link: geometry visual mesh filename=package://robot_description/meshes/robot3/rear_left_mount_l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
- link rear_left_wheel_link: geometry collision cylinder length=0.1000 radius=0.1749; visual mesh filename=package://robot_description/meshes/robot3/rear_left_wheel_l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
- link rear_right_motor_link: geometry visual mesh filename=package://robot_description/meshes/robot3/rear_right_motor_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
- link rear_right_mount_link: geometry visual mesh filename=package://robot_description/meshes/robot3/rear_right_mount_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
- link rear_right_wheel_link: geometry collision cylinder length=0.1000 radius=0.1749; visual mesh filename=package://robot_description/meshes/robot3/rear_right_wheel_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
Joints:
- removed joint front_left_motor_joint
- removed joint front_left_mount_joint
- removed joint front_left_wheel_joint
- removed joint front_right_motor_joint
- removed joint front_right_mount_joint
- removed joint front_right_wheel_joint
- added joint camera_mount_link_joint: type fixed, parent base_link, child camera_mount_link, origin xyz=0.2000 0.0000 0.7500 rpy=0.0000 0.0000 0.0000
- added joint front_left_caster_joint: type fixed, parent chassis, child front_left_caster_link, origin xyz=0.4682 0.5508 0.1222 rpy=0.0000 0.0000 0.0000
- added joint front_right_caster_joint: type fixed, parent chassis, child front_right_caster_link, origin xyz=0.4682 -0.5508 0.1222 rpy=0.0000 0.0000 0.0000
- added joint imu_0_link_joint: type fixed, parent base_link, child imu_0_link, origin xyz=0.0000 0.0000 0.3000 rpy=0.0000 0.0000 0.0000
- joint camera_0_link_joint: origin xyz=0.0000 0.0000 0.1000 rpy=0.0000 0.0000 0.0000 -> xyz=0.5750 0.5000 0.3100 rpy=0.0000 0.3100 0.0000
- joint rear_left_mount_joint: origin xyz=-0.4000 0.4742 0.2746 rpy=0.0000 0.0000 0.0000 -> xyz=-0.5246 0.4742 0.2746 rpy=0.0000 0.0000 0.0000
- joint rear_right_mount_joint: origin xyz=-0.4000 -0.4742 0.2746 rpy=0.0000 0.0000 0.0000 -> xyz=-0.5246 -0.4742 0.2746 rpy=0.0000 0.0000 0.0000

File: apps/robot/description/urdf/robot3/robot.urdf (robot description, URDF)
Before this commit: robot robot, 18 links, 17 joints
Links:
- removed link front_left_motor_link
- removed link front_left_mount_link
- removed link front_left_wheel_link
- removed link front_right_motor_link
- removed link front_right_mount_link
- removed link front_right_wheel_link
- added link camera_mount_link
- added link front_left_caster_link; collision sphere radius=0.1396
- added link front_right_caster_link; collision sphere radius=0.1396
- added link imu_0_link
- link chassis: geometry collision box size=1.2192 1.0000 0.0254; visual mesh filename=package://robot_description/meshes/robot3/chassis.dae
- link inertial_link: mass 41.2746 -> 63.6981
- link rear_left_motor_link: geometry visual mesh filename=package://robot_description/meshes/robot3/rear_left_motor_l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
- link rear_left_mount_link: geometry visual mesh filename=package://robot_description/meshes/robot3/rear_left_mount_l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
- link rear_left_wheel_link: geometry collision cylinder length=0.1000 radius=0.1749; visual mesh filename=package://robot_description/meshes/robot3/rear_left_wheel_l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
- link rear_right_motor_link: geometry visual mesh filename=package://robot_description/meshes/robot3/rear_right_motor_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
- link rear_right_mount_link: geometry visual mesh filename=package://robot_description/meshes/robot3/rear_right_mount_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
- link rear_right_wheel_link: geometry collision cylinder length=0.1000 radius=0.1749; visual mesh filename=package://robot_description/meshes/robot3/rear_right_wheel_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
Joints:
- removed joint front_left_motor_joint
- removed joint front_left_mount_joint
- removed joint front_left_wheel_joint
- removed joint front_right_motor_joint
- removed joint front_right_mount_joint
- removed joint front_right_wheel_joint
- added joint camera_mount_link_joint: type fixed, parent base_link, child camera_mount_link, origin xyz=0.2000 0.0000 0.7500 rpy=0.0000 0.0000 0.0000
- added joint front_left_caster_joint: type fixed, parent chassis, child front_left_caster_link, origin xyz=0.4682 0.5508 0.1222 rpy=0.0000 0.0000 0.0000
- added joint front_right_caster_joint: type fixed, parent chassis, child front_right_caster_link, origin xyz=0.4682 -0.5508 0.1222 rpy=0.0000 0.0000 0.0000
- added joint imu_0_link_joint: type fixed, parent base_link, child imu_0_link, origin xyz=0.0000 0.0000 0.3000 rpy=0.0000 0.0000 0.0000
- joint camera_0_link_joint: origin xyz=0.0000 0.0000 0.1000 rpy=0.0000 0.0000 0.0000 -> xyz=0.5750 0.5000 0.3100 rpy=0.0000 0.3100 0.0000
- joint rear_left_mount_joint: origin xyz=-0.4000 0.4742 0.2746 rpy=0.0000 0.0000 0.0000 -> xyz=-0.5246 0.4742 0.2746 rpy=0.0000 0.0000 0.0000
- joint rear_right_mount_joint: origin xyz=-0.4000 -0.4742 0.2746 rpy=0.0000 0.0000 0.0000 -> xyz=-0.5246 -0.4742 0.2746 rpy=0.0000 0.0000 0.0000
