Commit message: feat(robot/{description,generator_common,simulator): overhaul setup
Signed-off-by: Mumtahin Farabi <mfarabi619@gmail.com>

File: apps/robot/description/urdf/robot4/robot.sim.urdf (robot description, URDF)
Before this commit: robot robot, 18 links, 17 joints
Links:
- removed link camera_0_color_optical_frame
- removed link camera_0_link
- removed link front_left_motor_link
- removed link front_left_mount_link
- removed link front_left_wheel_link
- removed link front_right_motor_link
- removed link front_right_mount_link
- removed link front_right_wheel_link
- added link front_left_caster_link; collision sphere radius=0.1396
- added link front_right_caster_link; collision sphere radius=0.1396
- link chassis: geometry collision box size=1.2192 1.0000 0.0254; visual mesh filename=package://robot_description/meshes/robot4/chassis.dae
- link inertial_link: mass 41.2746 -> 63.6981
- link rear_left_motor_link: geometry visual mesh filename=package://robot_description/meshes/robot4/rear_left_motor_l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
- link rear_left_mount_link: geometry visual mesh filename=package://robot_description/meshes/robot4/rear_left_mount_l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
- link rear_left_wheel_link: geometry collision cylinder length=0.1000 radius=0.1749; visual mesh filename=package://robot_description/meshes/robot4/rear_left_wheel_l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
- link rear_right_motor_link: geometry visual mesh filename=package://robot_description/meshes/robot4/rear_right_motor_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
- link rear_right_mount_link: geometry visual mesh filename=package://robot_description/meshes/robot4/rear_right_mount_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
- link rear_right_wheel_link: geometry collision cylinder length=0.1000 radius=0.1749; visual mesh filename=package://robot_description/meshes/robot4/rear_right_wheel_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
Joints:
- removed joint camera_0_color_optical_frame_joint
- removed joint camera_0_link_joint
- removed joint front_left_motor_joint
- removed joint front_left_mount_joint
- removed joint front_left_wheel_joint
- removed joint front_right_motor_joint
- removed joint front_right_mount_joint
- removed joint front_right_wheel_joint
- added joint front_left_caster_joint: type fixed, parent chassis, child front_left_caster_link, origin xyz=0.4682 0.5508 0.1222 rpy=0.0000 0.0000 0.0000
- added joint front_right_caster_joint: type fixed, parent chassis, child front_right_caster_link, origin xyz=0.4682 -0.5508 0.1222 rpy=0.0000 0.0000 0.0000
- joint rear_left_mount_joint: origin xyz=-0.4000 0.4742 0.2746 rpy=0.0000 0.0000 0.0000 -> xyz=-0.5246 0.4742 0.2746 rpy=0.0000 0.0000 0.0000
- joint rear_right_mount_joint: origin xyz=-0.4000 -0.4742 0.2746 rpy=0.0000 0.0000 0.0000 -> xyz=-0.5246 -0.4742 0.2746 rpy=0.0000 0.0000 0.0000

File: apps/robot/description/urdf/robot5/robot.sim.urdf (robot description, URDF)
Before this commit: robot robot, 18 links, 17 joints
Links:
- removed link front_left_motor_link
- removed link front_left_mount_link
- removed link front_left_wheel_link
- removed link front_right_motor_link
- removed link front_right_mount_link
- removed link front_right_wheel_link
- added link front_left_caster_link; collision sphere radius=0.1396
- added link front_right_caster_link; collision sphere radius=0.1396
- link chassis: geometry collision box size=1.2192 1.0000 0.0254; visual mesh filename=package://robot_description/meshes/robot5/chassis.dae
- link inertial_link: mass 41.2746 -> 63.6981
- link rear_left_motor_link: geometry visual mesh filename=package://robot_description/meshes/robot5/rear_left_motor_l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
- link rear_left_mount_link: geometry visual mesh filename=package://robot_description/meshes/robot5/rear_left_mount_l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
- link rear_left_wheel_link: geometry collision cylinder length=0.1000 radius=0.1749; visual mesh filename=package://robot_description/meshes/robot5/rear_left_wheel_l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
- link rear_right_motor_link: geometry visual mesh filename=package://robot_description/meshes/robot5/rear_right_motor_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
- link rear_right_mount_link: geometry visual mesh filename=package://robot_description/meshes/robot5/rear_right_mount_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
- link rear_right_wheel_link: geometry collision cylinder length=0.1000 radius=0.1749; visual mesh filename=package://robot_description/meshes/robot5/rear_right_wheel_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
Joints:
- removed joint front_left_motor_joint
- removed joint front_left_mount_joint
- removed joint front_left_wheel_joint
- removed joint front_right_motor_joint
- removed joint front_right_mount_joint
- removed joint front_right_wheel_joint
- added joint front_left_caster_joint: type fixed, parent chassis, child front_left_caster_link, origin xyz=0.4682 0.5508 0.1222 rpy=0.0000 0.0000 0.0000
- added joint front_right_caster_joint: type fixed, parent chassis, child front_right_caster_link, origin xyz=0.4682 -0.5508 0.1222 rpy=0.0000 0.0000 0.0000
- joint rear_left_mount_joint: origin xyz=-0.4000 0.4742 0.2746 rpy=0.0000 0.0000 0.0000 -> xyz=-0.5246 0.4742 0.2746 rpy=0.0000 0.0000 0.0000
- joint rear_right_mount_joint: origin xyz=-0.4000 -0.4742 0.2746 rpy=0.0000 0.0000 0.0000 -> xyz=-0.5246 -0.4742 0.2746 rpy=0.0000 0.0000 0.0000

File: apps/robot/description/urdf/robot5/robot.urdf (robot description, URDF)
Before this commit: robot robot, 18 links, 17 joints
Links:
- removed link front_left_motor_link
- removed link front_left_mount_link
- removed link front_left_wheel_link
- removed link front_right_motor_link
- removed link front_right_mount_link
- removed link front_right_wheel_link
- added link front_left_caster_link; collision sphere radius=0.1396
- added link front_right_caster_link; collision sphere radius=0.1396
- link chassis: geometry collision box size=1.2192 1.0000 0.0254; visual mesh filename=package://robot_description/meshes/robot5/chassis.dae
- link inertial_link: mass 41.2746 -> 63.6981
- link rear_left_motor_link: geometry visual mesh filename=package://robot_description/meshes/robot5/rear_left_motor_l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
- link rear_left_mount_link: geometry visual mesh filename=package://robot_description/meshes/robot5/rear_left_mount_l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
- link rear_left_wheel_link: geometry collision cylinder length=0.1000 radius=0.1749; visual mesh filename=package://robot_description/meshes/robot5/rear_left_wheel_l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
- link rear_right_motor_link: geometry visual mesh filename=package://robot_description/meshes/robot5/rear_right_motor_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
- link rear_right_mount_link: geometry visual mesh filename=package://robot_description/meshes/robot5/rear_right_mount_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
- link rear_right_wheel_link: geometry collision cylinder length=0.1000 radius=0.1749; visual mesh filename=package://robot_description/meshes/robot5/rear_right_wheel_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
Joints:
- removed joint front_left_motor_joint
- removed joint front_left_mount_joint
- removed joint front_left_wheel_joint
- removed joint front_right_motor_joint
- removed joint front_right_mount_joint
- removed joint front_right_wheel_joint
- added joint front_left_caster_joint: type fixed, parent chassis, child front_left_caster_link, origin xyz=0.4682 0.5508 0.1222 rpy=0.0000 0.0000 0.0000
- added joint front_right_caster_joint: type fixed, parent chassis, child front_right_caster_link, origin xyz=0.4682 -0.5508 0.1222 rpy=0.0000 0.0000 0.0000
- joint rear_left_mount_joint: origin xyz=-0.4000 0.4742 0.2746 rpy=0.0000 0.0000 0.0000 -> xyz=-0.5246 0.4742 0.2746 rpy=0.0000 0.0000 0.0000
- joint rear_right_mount_joint: origin xyz=-0.4000 -0.4742 0.2746 rpy=0.0000 0.0000 0.0000 -> xyz=-0.5246 -0.4742 0.2746 rpy=0.0000 0.0000 0.0000

File: apps/robot/description/urdf/robot6/robot.sim.urdf (robot description, URDF)
Before this commit: robot robot, 12 links, 11 joints
Links:
- link chassis: geometry collision box size=1.2192 1.0000 0.0254; visual mesh filename=package://robot_description/meshes/robot6/chassis.dae
- link rear_left_motor_link: geometry visual mesh filename=package://robot_description/meshes/robot6/rear_left_motor_l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
- link rear_left_mount_link: geometry visual mesh filename=package://robot_description/meshes/robot6/rear_left_mount_l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
- link rear_left_wheel_link: geometry collision cylinder length=0.1000 radius=0.1749; visual mesh filename=package://robot_description/meshes/robot6/rear_left_wheel_l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
- link rear_right_motor_link: geometry visual mesh filename=package://robot_description/meshes/robot6/rear_right_motor_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
- link rear_right_mount_link: geometry visual mesh filename=package://robot_description/meshes/robot6/rear_right_mount_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
- link rear_right_wheel_link: geometry collision cylinder length=0.1000 radius=0.1749; visual mesh filename=package://robot_description/meshes/robot6/rear_right_wheel_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

File: apps/robot/description/urdf/robot6/robot.urdf (robot description, URDF)
Before this commit: robot robot, 12 links, 11 joints
Links:
- link chassis: geometry collision box size=1.2192 1.0000 0.0254; visual mesh filename=package://robot_description/meshes/robot6/chassis.dae
- link rear_left_motor_link: geometry visual mesh filename=package://robot_description/meshes/robot6/rear_left_motor_l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
- link rear_left_mount_link: geometry visual mesh filename=package://robot_description/meshes/robot6/rear_left_mount_l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
- link rear_left_wheel_link: geometry collision cylinder length=0.1000 radius=0.1749; visual mesh filename=package://robot_description/meshes/robot6/rear_left_wheel_l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
- link rear_right_motor_link: geometry visual mesh filename=package://robot_description/meshes/robot6/rear_right_motor_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
- link rear_right_mount_link: geometry visual mesh filename=package://robot_description/meshes/robot6/rear_right_mount_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
- link rear_right_wheel_link: geometry collision cylinder length=0.1000 radius=0.1749; visual mesh filename=package://robot_description/meshes/robot6/rear_right_wheel_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
