Commit message: feat(robot/mech): update setup and remove urdf topic collision
Signed-off-by: Mumtahin Farabi <mfarabi619@gmail.com>

File: apps/robot/mech/urdf/robot2/robot.sim.urdf (robot description, URDF)
Before this commit: robot robot, 14 links, 13 joints
Links:
- link inertial_link: mass 63.6981 -> 58.0389

File: apps/robot/mech/urdf/robot2/robot.urdf (robot description, URDF)
Before this commit: robot robot, 14 links, 13 joints
Links:
- link inertial_link: mass 63.6981 -> 58.0389

File: apps/robot/mech/urdf/robot3/robot.sim.urdf (robot description, URDF)
Before this commit: robot robot, 16 links, 15 joints
Links:
- link inertial_link: mass 63.6981 -> 58.0389

File: apps/robot/mech/urdf/robot3/robot.urdf (robot description, URDF)
Before this commit: robot robot, 16 links, 15 joints
Links:
- link inertial_link: mass 63.6981 -> 58.0389

File: apps/robot/mech/urdf/robot4/robot.sim.urdf (robot description, URDF)
Before this commit: robot robot, 12 links, 11 joints
Links:
- link inertial_link: mass 63.6981 -> 58.0389

File: apps/robot/mech/urdf/robot4/robot.urdf (robot description, URDF)
Before this commit: robot robot, 12 links, 11 joints
Links:
- link inertial_link: mass 63.6981 -> 58.0389

File: apps/robot/mech/urdf/robot5/robot.sim.urdf (robot description, URDF)
Before this commit: robot robot, 14 links, 13 joints
Links:
- link inertial_link: mass 63.6981 -> 58.0389

File: apps/robot/mech/urdf/robot5/robot.urdf (robot description, URDF)
Before this commit: robot robot, 14 links, 13 joints
Links:
- link inertial_link: mass 63.6981 -> 58.0389

File: apps/robot/mech/urdf/robot6/robot.sim.urdf (robot description, URDF)
Before this commit: robot robot, 12 links, 11 joints
Links:
- link inertial_link: mass 63.6981 -> 58.0389

File: apps/robot/mech/urdf/robot6/robot.urdf (robot description, URDF)
Before this commit: robot robot, 12 links, 11 joints
Links:
- link inertial_link: mass 63.6981 -> 58.0389

File: apps/robot/mech/urdf/taro/robot.sim.urdf (robot description, URDF)
Before this commit: robot robot, 14 links, 13 joints
Links:
- link inertial_link: mass 63.6981 -> 58.0389
Joints:
- joint camera_0_link_joint: origin xyz=0.5300 0.4750 0.5660 rpy=0.0000 0.0000 0.0000 -> xyz=0.5300 0.4750 0.4690 rpy=0.0000 0.0000 0.0000

File: apps/robot/mech/urdf/taro/robot.urdf (robot description, URDF)
Before this commit: robot robot, 14 links, 13 joints
Links:
- link inertial_link: mass 63.6981 -> 58.0389
Joints:
- joint camera_0_link_joint: origin xyz=0.5300 0.4750 0.5660 rpy=0.0000 0.0000 0.0000 -> xyz=0.5300 0.4750 0.4690 rpy=0.0000 0.0000 0.0000
