Commit message: feat(robot/mech): add caster wheel kinematics
Signed-off-by: Mumtahin Farabi <mfarabi619@gmail.com>

File: apps/robot/mech/urdf/jiro/robot.sim.urdf (robot description, URDF)
Before this commit: robot robot, 14 links, 13 joints
Links:
- link front_left_caster_link: geometry collision cylinder length=0.1000 radius=0.1396
- link front_right_caster_link: geometry collision cylinder length=0.1000 radius=0.1396

File: apps/robot/mech/urdf/robot2/robot.sim.urdf (robot description, URDF)
Before this commit: robot robot, 14 links, 13 joints
Links:
- link front_left_caster_link: geometry collision cylinder length=0.1000 radius=0.1396
- link front_right_caster_link: geometry collision cylinder length=0.1000 radius=0.1396

File: apps/robot/mech/urdf/robot3/robot.sim.urdf (robot description, URDF)
Before this commit: robot robot, 16 links, 15 joints
Links:
- link front_left_caster_link: geometry collision cylinder length=0.1000 radius=0.1396
- link front_right_caster_link: geometry collision cylinder length=0.1000 radius=0.1396

File: apps/robot/mech/urdf/robot4/robot.sim.urdf (robot description, URDF)
Before this commit: robot robot, 12 links, 11 joints
Links:
- link front_left_caster_link: geometry collision cylinder length=0.1000 radius=0.1396
- link front_right_caster_link: geometry collision cylinder length=0.1000 radius=0.1396

File: apps/robot/mech/urdf/robot5/robot.sim.urdf (robot description, URDF)
Before this commit: robot robot, 14 links, 13 joints
Links:
- link front_left_caster_link: geometry collision cylinder length=0.1000 radius=0.1396
- link front_right_caster_link: geometry collision cylinder length=0.1000 radius=0.1396

File: apps/robot/mech/urdf/robot6/robot.sim.urdf (robot description, URDF)
Before this commit: robot robot, 12 links, 11 joints
Links:
- link front_left_caster_link: geometry collision cylinder length=0.1000 radius=0.1396
- link front_right_caster_link: geometry collision cylinder length=0.1000 radius=0.1396

File: apps/robot/mech/urdf/taro/robot.sim.urdf (robot description, URDF)
Before this commit: robot robot, 14 links, 13 joints
Links:
- added link gps_link
- link front_left_caster_link: geometry collision cylinder length=0.1000 radius=0.1396
- link front_right_caster_link: geometry collision cylinder length=0.1000 radius=0.1396
Joints:
- added joint gps_link_joint: type fixed, parent base_link, child gps_link, origin xyz=0.0000 0.0000 0.0000 rpy=0.0000 0.0000 0.0000

File: apps/robot/mech/urdf/taro/robot.urdf (robot description, URDF)
Before this commit: robot robot, 14 links, 13 joints
Links:
- added link gps_link
Joints:
- added joint gps_link_joint: type fixed, parent base_link, child gps_link, origin xyz=0.0000 0.0000 0.0000 rpy=0.0000 0.0000 0.0000
