Commit message: feat(robot/driver/roboteq): scaffold setup
Signed-off-by: Mumtahin Farabi <mfarabi619@gmail.com>

File: apps/robot/mech/urdf/robot7/robot.sim.urdf (robot description, URDF)
Before this commit: robot robot, 14 links, 13 joints
Links:
- removed link camera_0_color_optical_frame
- removed link camera_0_link
- link chassis: geometry collision box size=1.2192 1.0000 0.0254; visual mesh filename=package://robot_description/meshes/robot7/chassis.dae
- link rear_left_motor_link: geometry visual mesh filename=package://robot_description/meshes/robot7/rear_left_motor_l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
- link rear_left_mount_link: geometry visual mesh filename=package://robot_description/meshes/robot7/rear_left_mount_l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
- link rear_left_wheel_link: geometry collision cylinder length=0.1000 radius=0.1749; visual mesh filename=package://robot_description/meshes/robot7/rear_left_wheel_l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
- link rear_right_motor_link: geometry visual mesh filename=package://robot_description/meshes/robot7/rear_right_motor_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
- link rear_right_mount_link: geometry visual mesh filename=package://robot_description/meshes/robot7/rear_right_mount_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
- link rear_right_wheel_link: geometry collision cylinder length=0.1000 radius=0.1749; visual mesh filename=package://robot_description/meshes/robot7/rear_right_wheel_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
Joints:
- removed joint camera_0_color_optical_frame_joint
- removed joint camera_0_link_joint

File: apps/robot/mech/urdf/robot7/robot.urdf (robot description, URDF)
Before this commit: robot robot, 14 links, 13 joints
Links:
- removed link camera_0_color_optical_frame
- removed link camera_0_link
- link chassis: geometry collision box size=1.2192 1.0000 0.0254; visual mesh filename=package://robot_description/meshes/robot7/chassis.dae
- link front_left_caster_link: geometry 
- link front_right_caster_link: geometry 
- link rear_left_motor_link: geometry visual mesh filename=package://robot_description/meshes/robot7/rear_left_motor_l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
- link rear_left_mount_link: geometry visual mesh filename=package://robot_description/meshes/robot7/rear_left_mount_l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
- link rear_left_wheel_link: geometry collision cylinder length=0.1000 radius=0.1749; visual mesh filename=package://robot_description/meshes/robot7/rear_left_wheel_l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
- link rear_right_motor_link: geometry visual mesh filename=package://robot_description/meshes/robot7/rear_right_motor_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
- link rear_right_mount_link: geometry visual mesh filename=package://robot_description/meshes/robot7/rear_right_mount_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
- link rear_right_wheel_link: geometry collision cylinder length=0.1000 radius=0.1749; visual mesh filename=package://robot_description/meshes/robot7/rear_right_wheel_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
Joints:
- removed joint camera_0_color_optical_frame_joint
- removed joint camera_0_link_joint
