Commit message: feat(robot/manipulation): overhaul setup
Signed-off-by: Mumtahin Farabi <mfarabi619@gmail.com>

File: apps/robot/mech/urdf/kinova-link-6/robot.sim.urdf (robot description, URDF)
Before this commit: robot link6, 18 links, 17 joints
Links:
- added link controller_link; visual mesh filename=package://robot_description/urdf/kinova-link-6/meshes/contr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 scale=0.001 0.001 0.001; visual mesh filename=package://robot_description/urdf/kinova-link-6/meshes/penda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 scale=0.001 0.001 0.001
- added link flange_adapter_link; visual mesh filename=package://robot_description/urdf/kinova-link-6/meshes/flang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 scale=0.001 0.001 0.001
- added link gripper_mount_link
Joints:
- added joint controller_joint: type fixed, parent base_link, child controller_link, origin xyz=0 0 0 rpy=0 0 0
- added joint flange_adapter_joint: type fixed, parent end_effector_link, child flange_adapter_link, origin xyz=0 0 0 rpy=0 0 0
- added joint gripper_mount_joint: type fixed, parent flange_adapter_link, child gripper_mount_link, origin xyz=0 0 0.0265 rpy=0 0 0
- joint robotiq_85_base_joint: parent end_effector_link -> gripper_mount_link

File: apps/robot/mech/urdf/kinova-link-6/robot.urdf (robot description, URDF)
Before this commit: robot link6, 18 links, 17 joints
Links:
- added link controller_link; visual mesh filename=package://robot_description/urdf/kinova-link-6/meshes/contr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 scale=0.001 0.001 0.001; visual mesh filename=package://robot_description/urdf/kinova-link-6/meshes/penda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 scale=0.001 0.001 0.001
- added link flange_adapter_link; visual mesh filename=package://robot_description/urdf/kinova-link-6/meshes/flang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 scale=0.001 0.001 0.001
- added link gripper_mount_link
Joints:
- added joint controller_joint: type fixed, parent base_link, child controller_link, origin xyz=0 0 0 rpy=0 0 0
- added joint flange_adapter_joint: type fixed, parent end_effector_link, child flange_adapter_link, origin xyz=0 0 0 rpy=0 0 0
- added joint gripper_mount_joint: type fixed, parent flange_adapter_link, child gripper_mount_link, origin xyz=0 0 0.0265 rpy=0 0 0
- joint robotiq_85_base_joint: parent end_effector_link -> gripper_mount_link
